File: pcb/alpha_1.4/ogn_wind_1.4.brd (EAGLE design)
At the start: 56.3 x 23.9 mm, 67 parts, among them IC1 CN3791, IC2 BMP280, IC3 MCP4652T-104E_MF, IC4 TPS22975DSGT, J1 CON-SMA-EDGE-S, J4 CONSMA001-SMD-G, Q1 PMPB16EPX, Q2 PMPB16EPX, SW1 SPST_TACT-KMR2, U1 MT3608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

Commit message: mini V2.0
Parts:
- added ANT_UFL: (no value), ufl:U.FL
Connections:
- net ANT: now also ANT_UFL.P$3
- net GND: now also ANT_UFL.P$1, ANT_UFL.P$2, ANT_UFL.P$4
