File: pcb/alpha_1.4/ogn_wind_1.4.sch (EAGLE design)
At the start: 67 parts, among them IC1 CN3791, IC2 BMP280, IC3 MCP4652T-104E_MF, IC4 TPS22975DSGT, J1 CON-SMA-EDGE-S, J4 CONSMA001-SMD-G, Q1 PMPB16EPX, Q2 PMPB16EPX, SW1 SPST_TACT-KMR2, U1 MT3608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

Commit message: mini V2.0
Parts:
- added ANT_UFL: (no value), ufl:U.FL
Connections:
- net ANT: now also ANT_UFL.SIGNAL
- net GND: now also ANT_UFL.GND@0, ANT_UFL.GND@1, ANT_UFL.GND@2
Changed lines of the file:
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@@
 <layer number="135" name="BGA_NC" color="7" fill="1" visible="yes" active="yes"/>
 <layer number="136" name="BGA_DED" color="7" fill="1" visible="yes" active="yes"/>
+<layer number="137" name="silkbottom" color="7" fill="1" visible="yes" active="yes"/>
+<layer number="138" name="EEE" color="7" fill="1" visible="yes" active="yes"/>
+<layer number="139" name="_tKeepout" color="7" fill="1" visible="yes" active="yes"/>
+<layer number="140" name="mbKeepout" color="7" fill="1" visible="yes" active="yes"/>
+<layer number="141" name="ASSEMBLY_TOP" color="7" fill="1" visible="yes" active="yes"/>
+<layer number="142" name="mbRestrict" color="7" fill="1" visible="yes" active="yes"/>
+<layer number="143" name="PLACE_BOUND_TOP" color="7" fill="1" visible="yes" active="yes"/>
 <layer number="144" name="Drill_legend" color="7" fill="1" visible="no" active="yes"/>
 <layer number="145" name="DrillLegend_01-02" color="7" fill="1" visible="yes" active="yes"/>
@@
 <layer number="154" name="FabDoc2" color="2" fill="1" visible="no" active="no"/>
 <layer number="155" name="FabDoc3" color="7" fill="15" visible="no" active="no"/>
+<layer number="166" name="AntennaArea" color="7" fill="1" visible="yes" active="yes"/>
+<layer number="168" name="4mmHeightArea" color="7" fill="1" visible="yes" active="yes"/>
+<layer number="191" name="mNets" color="7" fill="1" visible="yes" active="yes"/>
+<layer number="192" name="mBusses" color="7" fill="1" visible="yes" active="yes"/>
+<layer number="193" name="mPins" color="7" fill="1" visible="yes" active="yes"/>
+<layer number="194" name="mSymbols" color="7" fill="1" visible="yes" active="yes"/>
+<layer number="195" name="mNames" color="7" fill="1" visible="yes" active="yes"/>
+<layer number="196" name="mValues" color="7" fill="1" visible="yes" active="yes"/>
 <layer number="199" name="Contour" color="7" fill="1" visible="no" active="yes"/>
 <layer number="200" name="200bmp" color="1" fill="10" visible="no" active="yes"/>
@@
 </part>
 <part name="U$22" library="000_eigene_Bauteile" deviceset="SJ" device=""/>
+<part name="ANT_UFL" library="ufl" deviceset="U.FL" device=""/>
 </parts>
 <sheets>
@@
 </instance>
 <instance part="U$22" gate="G$1" x="137.16" y="-55.88" smashed="yes"/>
+<instance part="ANT_UFL" gate="G$1" x="160.02" y="-63.5" smashed="yes"/>
 </instances>
 <busses>
@@
 <wire x1="116.84" y1="55.88" x2="114.3" y2="55.88" width="0.1524" layer="91"/>
 <label x="114.3" y="55.88" size="1.27" layer="95" rot="R180" xref="yes"/>
+</segment>
+<segment>
+<pinref part="ANT_UFL" gate="G$1" pin="GND@0"/>
+<pinref part="ANT_UFL" gate="G$1" pin="GND@1"/>
+<wire x1="154.94" y1="-71.12" x2="157.48" y2="-71.12" width="0.1524" layer="91"/>
+<wire x1="157.48" y1="-71.12" x2="157.48" y2="-68.58" width="0.1524" layer="91"/>
+<junction x="157.48" y="-71.12"/>
+<pinref part="ANT_UFL" gate="G$1" pin="GND@2"/>
+<wire x1="157.48" y1="-73.66" x2="157.48" y2="-71.12" width="0.1524" layer="91"/>
+<label x="154.94" y="-71.12" size="1.27" layer="95" rot="R180" xref="yes"/>
 </segment>
 </net>
@@
 <pinref part="U$22" gate="G$1" pin="P$2"/>
 </segment>
-</net>
+<segment>
+<pinref part="ANT_UFL" gate="G$1" pin="SIGNAL"/>
+<wire x1="165.1" y1="-63.5" x2="167.64" y2="-63.5" width="0.1524" layer="91"/>
+<label x="167.64" y="-63.5" size="1.27" layer="95" xref="yes"/>
+</segment>
+</net>
